Commit message: set proper rotation of imu frame

File: urdf/robot.urdf.xacro (robot description, xacro)
@@ -88,5 +88,5 @@
   </xacro:sensor_d435>
   <joint name="imu_joint" type="fixed">
-    <origin xyz="0 0.0762 0.004" rpy="0 0 0" />
+    <origin xyz="0 0.0762 0.004" rpy="3.14 0.0 0.0" />
     <parent link="hoop_link" />
     <child link="imu_link" />

Commit message: cleanup package.xml and urdf

File: urdf/robot.urdf.xacro (robot description, xacro)
@@ -1,5 +1,4 @@
 <?xml version="1.0"?>
 <robot xmlns:xacro="http://www.ros.org/wiki/xacro" name="robomagellan">
-  <xacro:include filename="$(find realsense2_description)/urdf/_d435.urdf.xacro" />
   <material name="black">
     <color rgba="0.1 0.1 0.1 1.0" />
@@ -83,8 +82,4 @@
     </visual>
   </link>
-  <!-- Camera -->
-  <xacro:sensor_d435 parent="camera_mount">
-    <origin xyz="0.038 0 -0.022" rpy="0 0.349 0"/>
-  </xacro:sensor_d435>
   <joint name="imu_joint" type="fixed">
     <origin xyz="0 0.0762 0.004" rpy="3.14 0.0 0.0" />
